File: Embedded/AC_Logger/HW/AFE_Board/AFE_Board.kicad_pcb (KiCad board)
At the start: 2 copper layers, 111.8 x 88.9 mm, 58 parts, among them J1 Screw_Terminal_01x02, J2 Screw_Terminal_01x02, J3 Screw_Terminal_01x02, J4 Screw_Terminal_01x02, J5 Conn_01x04, J6 Conn_01x06, J7 Conn_01x04, J8 NS25-W3P male, T1 ASM-010, T2 ASM-010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

Commit message: Corrections.
Parts:
- moved J8 15.2 mm to (124.5, 25.4)
Routing:
- net VEE: track 238.8 -> 243.8 mm
- net GND: track 448.8 -> 453.9 mm
