File: Embedded/AC_Logger/HW/Unnulling_Board_v2/Unnulling_Board.kicad_pcb (KiCad board)
At the start: 2 copper layers, 58.4 x 61 mm, 18 parts, among them J1 Screw_Terminal_01x03, J2 Screw_Terminal_01x04, K1 RT424048, K2 RT424048

Commit message: Final v2
Parts:
- removed C1, C2: 220n 310V X2, Capacitor_THT:C_Rect_L16.5mm_W8.7mm_P15.00mm_MKT
- D1, D2: footprint Diode_THT:D_DO-41_SOD81_P7.62mm_Horizontal -> For_Rasterboard:D_DO-35_SOD27_Pinf_Horizontal
- R1, R2: value 100 1W -> 10k 1W
- moved D2 13.3 mm to (53.3, 78.7), turned to 90 degrees
- moved D5 11.4 mm to (88.9, 76.2)
- moved C4 11.4 mm to (81.3, 76.2)
- moved K1 11.4 mm to (88.8, 68.5)
- moved R1 10.5 mm to (86.4, 88.9)
- moved J2 10.5 mm to (99.1, 66.0), turned to 90 degrees
- moved C3 10.5 mm to (61.0, 76.2)
- moved D3 10.5 mm to (68.6, 76.2)
- moved K2 10.5 mm to (68.5, 68.5)
- moved D1 10.2 mm to (76.2, 77.5), turned to 90 degrees
- moved R2 8.13 mm to (66.0, 88.9)
- moved J1 2.54 mm to (45.7, 63.5)
Connections:
- D1 pad 2: Net-(D1-A) -> /L1_OR_R3_IN
- D2 pad 2: Net-(D2-A) -> /N_IN
- J1 pad 1: /E -> /L1_OR_R3_IN
- J1 pad 2: /L1_OR_R3_IN -> /N_IN
- J1 pad 3: /N_IN -> /E
Routing:
- net /N_IN: track 0.00 -> 78.7 mm, vias 0 -> 3
- net /L1_OR_R3: track 28.0 -> 63.3 mm, vias 0 -> 2
- net /L1_OR_R3_IN: track 38.5 -> 70.0 mm, vias 0 -> 3
- net Net-(D2-K): track 0.00 -> 22.9 mm, vias 0 -> 1
- net Net-(D1-K): track 0.00 -> 21.6 mm, vias 0 -> 1
- net /unnulling/CTRL_WRONG: track 5.10 -> 25.5 mm, vias 1 -> 2
- net /E: track 38.3 -> 53.6 mm
- net /N: track 30.9 -> 40.8 mm
- net /unnulling/CTRL_CORRECT: track 21.4 -> 25.5 mm
Other:
- board size 58.4 x 61 mm -> 58.4 x 55.9 mm
