File: Embedded/AC_Logger/HW/Unnulling_Board_v2/Unnulling_Board.kicad_sch (KiCad schematic)
At the start: 6 parts, among them J1 Screw_Terminal_01x03, J2 Screw_Terminal_01x04

Commit message: Final v2
Connections:
- net E: now also J1.3 (Pin_3); no longer J1.1 (Pin_1)
- net L1_OR_R3_IN: now also J1.1 (Pin_1); no longer J1.2 (Pin_2)
- net N_IN: now also J1.2 (Pin_2); no longer J1.3 (Pin_3)
Changed lines of the file:
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@@
 	)
 	(label "L1_OR_R3_IN"
+		(at 106.68 78.74 180)
+		(effects
+			(font
+				(size 1.27 1.27)
+			)
+			(justify right bottom)
+		)
+	)
+	(label "N_IN"
 		(at 106.68 81.28 180)
 		(effects
@@
 		)
 	)
-	(label "N_IN"
+	(label "E"
 		(at 106.68 83.82 180)
 		(effects
 			(font
-				(size 1.27 1.27)
-			)
-			(justify right bottom)
-		)
-	)
-	(label "E"
-		(at 106.68 78.74 180)
-		(effects
-			(font
