File: Embedded/AC_Logger/HW/Unnulling_v2/Unnulling.kicad_sch (KiCad schematic)
At the start: 12 parts, among them K1 RT424048, K2 RT424048

Commit message: Final v2
Parts:
- removed C1, C2: 220n 310V X2, Capacitor_THT:C_Rect_L16.5mm_W8.7mm_P15.00mm_MKT, symbol Device:C
- D1, D2: footprint Diode_THT:D_DO-41_SOD81_P7.62mm_Horizontal -> For_Rasterboard:D_DO-35_SOD27_Pinf_Horizontal
- R1, R2: value 100 1W -> 10k 1W
Connections:
- net L1_OR_R3_IN: now also D1.2 (A)
- net N_IN: now also D2.2 (A)
Changed lines of the file:
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@@
 	(wire
 		(pts
-			(xy 25.4 125.73) (xy 44.45 125.73)
-		)
-		(stroke
-			(width 0)
-			(type default)
-		)
-	)
-	(wire
-		(pts
-			(xy 22.86 82.55) (xy 41.91 82.55)
+			(xy 36.83 125.73) (xy 55.88 125.73)
+		)
+		(stroke
+			(width 0)
+			(type default)
+		)
+	)
+	(wire
+		(pts
+			(xy 34.29 82.55) (xy 53.34 82.55)
 		)
 		(stroke
@@
 		(pts
 			(xy 170.18 106.68) (xy 157.48 106.68)
-		)
-		(stroke
-			(width 0)
-			(type default)
-		)
-	)
-	(wire
-		(pts
-			(xy 49.53 82.55) (xy 53.34 82.55)
-		)
-		(stroke
-			(width 0)
-			(type default)
-		)
-	)
-	(wire
-		(pts
-			(xy 52.07 125.73) (xy 55.88 125.73)
 		)
 		(stroke
@@
 	)
 	(label "L1_OR_R3_IN"
-		(at 38.1 82.55 180)
+		(at 49.53 82.55 180)
 		(effects
 			(font
@@
 	)
 	(label "N_IN"
-		(at 39.37 125.73 180)
+		(at 50.8 125.73 180)
 		(effects
 			(font
@@
 	(hierarchical_label "L1_OR_R3_IN"
 		(shape input)
-		(at 22.86 82.55 180)
+		(at 34.29 82.55 180)
 		(effects
 			(font
@@
 	(hierarchical_label "N_IN"
 		(shape input)
-		(at 25.4 125.73 180)
+		(at 36.83 125.73 180)
 		(effects
 			(font
@@
 	(hierarchical_label "E"
 		(shape input)
-		(at 34.29 101.6 180)
+		(at 33.02 101.6 180)
 		(effects
 			(font
@@
 			)
 		)
-		(property "Value" "100 1W"
+		(property "Value" "10k 1W"
 			(at 67.31 78.74 90)
 			(effects
@@
 	)
 	(symbol
-		(lib_id "Device:C")
-		(at 48.26 125.73 90)
-		(unit 1)
-		(exclude_from_sim no)
-		(in_bom yes)
-		(on_board yes)
-		(dnp no)
-		(fields_autoplaced yes)
-		(property "Reference" "C2"
-			(at 48.26 118.11 90)
-			(effects
-				(font
-					(size 1.27 1.27)
-				)
-			)
-		)
-		(property "Value" "220n 310V X2"
-			(at 48.26 120.65 90)
-			(effects
-				(font
-					(size 1.27 1.27)
-				)
-			)
-		)
-		(property "Footprint" "Capacitor_THT:C_Rect_L16.5mm_W8.7mm_P15.00mm_MKT"
-			(at 52.07 124.7648 0)
-			(effects
-				(font
-					(size 1.27 1.27)
-				)
-				(hide yes)
-			)
-		)
-		(property "Datasheet" "~"
-			(at 48.26 125.73 0)
-			(effects
-				(font
-					(size 1.27 1.27)
-				)
-				(hide yes)
-			)
-		)
-		(property "Description" "Unpolarized capacitor"
-			(at 48.26 125.73 0)
-			(effects
-				(font
-					(size 1.27 1.27)
-				)
-				(hide yes)
-			)
-		)
-		(pin "1"
-		)
-		(pin "2"
-		)
-		(instances
-			(project "Unnulling_Board"
-				(path "/496f50f6-b2f3-4b8a-9f23-d0b8419323e8/2b83cf42-630a-4dc0-9357-07fac29e3f84"
-					(reference "C2")
-					(unit 1)
-				)
-			)
-		)
-	)
-	(symbol
 		(lib_id "Device:R")
 		(at 69.85 125.73 90)
@@
 			)
 		)
-		(property "Value" "100 1W"
+		(property "Value" "10k 1W"
 			(at 69.85 121.92 90)
 			(effects
@@
 				(path "/496f50f6-b2f3-4b8a-9f23-d0b8419323e8/2b83cf42-630a-4dc0-9357-07fac29e3f84"
 					(reference "R2")
-					(unit 1)
-				)
-			)
-		)
-	)
-	(symbol
-		(lib_id "Device:C")
-		(at 45.72 82.55 90)
-		(unit 1)
-		(exclude_from_sim no)
-		(in_bom yes)
-		(on_board yes)
-		(dnp no)
-		(fields_autoplaced yes)
-		(property "Reference" "C1"
-			(at 45.72 74.93 90)
-			(effects
-				(font
-					(size 1.27 1.27)
-				)
-			)
-		)
-		(property "Value" "220n 310V X2"
-			(at 45.72 77.47 90)
-			(effects
-				(font
-					(size 1.27 1.27)
-				)
-			)
-		)
-		(property "Footprint" "Capacitor_THT:C_Rect_L16.5mm_W8.7mm_P15.00mm_MKT"
-			(at 49.53 81.5848 0)
-			(effects
-				(font
-					(size 1.27 1.27)
-				)
-				(hide yes)
-			)
-		)
-		(property "Datasheet" "~"
-			(at 45.72 82.55 0)
-			(effects
-				(font
-					(size 1.27 1.27)
-				)
-				(hide yes)
-			)
-		)
-		(property "Description" "Unpolarized capacitor"
-			(at 45.72 82.55 0)
-			(effects
-				(font
-					(size 1.27 1.27)
-				)
-				(hide yes)
-			)
-		)
-		(pin "1"
-		)
-		(pin "2"
-		)
-		(instances
-			(project ""
-				(path "/496f50f6-b2f3-4b8a-9f23-d0b8419323e8/2b83cf42-630a-4dc0-9357-07fac29e3f84"
-					(reference "C1")
 					(unit 1)
 				)
@@
 			)
 		)
-		(property "Footprint" "Diode_THT:D_DO-41_SOD81_P7.62mm_Horizontal"
+		(property "Footprint" "For_Rasterboard:D_DO-35_SOD27_Pinf_Horizontal"
 			(at 59.69 121.285 0)
 			(effects
@@
 			)
 		)
-		(property "Footprint" "Diode_THT:D_DO-41_SOD81_P7.62mm_Horizontal"
+		(property "Footprint" "For_Rasterboard:D_DO-35_SOD27_Pinf_Horizontal"
 			(at 57.15 78.105 0)
 			(effects
